File: FCOMMS_AD9361/FCOMMS_AD9361.kicad_pcb (KiCad board)
At the start: 8 copper layers, 200 x 125 mm, 47 parts, among them J301 Conn_Coaxial, J302 Conn_Coaxial, J303 Conn_Coaxial, J304 Conn_Coaxial, U201 LT8644SIV-TRMPBF, U301 AD9361BBCZ

Commit message: agile RF
Parts:
- removed C1001, C1003: 4.7uF, Capacitor_SMD:C_0603_1608Metric
- removed C1002, C903: 1nF, Capacitor_SMD:C_0603_1608Metric
- removed R1001, R902: 100k, Resistor_SMD:R_0603_1608Metric
- removed R1002, R901: 16K, Resistor_SMD:R_0603_1608Metric
- removed R1003, R903: 10K, Resistor_SMD:R_0603_1608Metric
- removed TP301, TP302, TP303, TP304: TestPoint, TestPoint:TestPoint_Pad_D1.0mm
- added C204: 22µF, Capacitor_SMD:C_0603_1608Metric, F.Cu at (216.3, 107.7)
- added C205: 8200pF, Capacitor_SMD:C_0603_1608Metric, F.Cu at (222.8, 115.7)
- added C212: 0.01µF, Capacitor_SMD:C_0805_2012Metric, F.Cu at (142.5, 97.0)
- added C213: 0.01µF, Capacitor_SMD:C_0805_2012Metric, F.Cu at (149.0, 97.0)
- added C214: 0.01µF, Capacitor_SMD:C_0805_2012Metric, F.Cu at (151.0, 97.0)
- added C215: C, Capacitor_SMD:C_0603_1608Metric, F.Cu at (228.0, 113.5)
- added C216: 4.7uF, Capacitor_SMD:C_0805_2012Metric, F.Cu at (207.7, 81.4)
- added C217: 100µF, Capacitor_SMD:C_1206_3216Metric, F.Cu at (217.5, 103.0)
- added C218: 100µF, Capacitor_SMD:C_1206_3216Metric, F.Cu at (225.8, 103.0)
- added C219: 0.15µF, Capacitor_SMD:C_0603_1608Metric, F.Cu at (215.5, 102.3)
- added C220: 0.15µF, Capacitor_SMD:C_0603_1608Metric, F.Cu at (227.8, 102.3)
- added C221: 1nF, Capacitor_SMD:C_0603_1608Metric, F.Cu at (202.2, 75.4)
- added C222: C, Capacitor_SMD:C_0603_1608Metric, F.Cu at (228.0, 116.5)
- added C223: 4.7uF, Capacitor_SMD:C_0805_2012Metric, F.Cu at (199.0, 84.0)
- added C224: 4.7uF, Capacitor_SMD:C_0805_2012Metric, F.Cu at (203.0, 84.0)
- added C225: 0.1 µF, Capacitor_SMD:C_0603_1608Metric, F.Cu at (199.4, 86.0)
- added C226: 0.1 µF, Capacitor_SMD:C_0603_1608Metric, F.Cu at (202.4, 86.0)
- added C227: 0.1µF, Capacitor_SMD:C_0603_1608Metric, F.Cu at (202.4, 87.5)
- added C228: 0.1 µF, Capacitor_SMD:C_0603_1608Metric, F.Cu at (199.4, 87.5)
- added C229: 4.7uF, Capacitor_SMD:C_0805_2012Metric, F.Cu at (206.3, 103.1)
- added C230: 1nF, Capacitor_SMD:C_0603_1608Metric, F.Cu at (221.3, 115.7)
- added C231: 1nF, Capacitor_SMD:C_0603_1608Metric, F.Cu at (201.8, 97.9)
- added C232: 4.7uF, Capacitor_SMD:C_0805_2012Metric, F.Cu at (198.5, 107.1)
- added C233: 4.7uF, Capacitor_SMD:C_0805_2012Metric, F.Cu at (201.9, 107.1)
- added C234: 0.1 µF, Capacitor_SMD:C_0603_1608Metric, F.Cu at (201.8, 109.1)
- added C235: 0.1 µF, Capacitor_SMD:C_0603_1608Metric, F.Cu at (198.8, 109.1)
- added C236: 0.1 µF, Capacitor_SMD:C_0603_1608Metric, F.Cu at (201.8, 110.6)
- added C237: 0.1 µF, Capacitor_SMD:C_0603_1608Metric, F.Cu at (198.8, 110.6)
- added C301: 18pF, Capacitor_SMD:C_0603_1608Metric, F.Cu at (64.2, 93.7)
- added C302: 18pF, Capacitor_SMD:C_0603_1608Metric, F.Cu at (64.2, 92.2)
- added C303: 18pF, Capacitor_SMD:C_0603_1608Metric, F.Cu at (90.0, 58.0)
- added C304: 18pF, Capacitor_SMD:C_0603_1608Metric, F.Cu at (91.5, 58.0)
- added C311: 12pF, Capacitor_SMD:C_0603_1608Metric, F.Cu at (102.4, 79.1)
- added C312: 12 pF, Capacitor_SMD:C_0603_1608Metric, F.Cu at (97.9, 79.3)
- added C601: 0.001µF, Capacitor_SMD:C_0603_1608Metric, F.Cu at (60.9, 47.8)
- added C602: 10 µF, Capacitor_SMD:C_0603_1608Metric, F.Cu at (59.4, 47.8)
- added C801: 22uF, Capacitor_SMD:C_0603_1608Metric, F.Cu at (246.3, 102.5)
- added C802: 68uF, Capacitor_SMD:C_1206_3216Metric, F.Cu at (238.8, 99.0)
- added C803: 22uF, Capacitor_SMD:C_0603_1608Metric, F.Cu at (246.3, 98.5)
- added FB201: 75 Ohms @ 100 MHz, Inductor_SMD:L_0603_1608Metric, F.Cu at (138.5, 99.5)
- added FB202: 30 Ohms @ 100 MHz, Inductor_SMD:L_0603_1608Metric, F.Cu at (147.0, 100.0)
- added FB203: 30 Ohms @ 100 MHz, Inductor_SMD:L_0603_1608Metric, F.Cu at (202.4, 89.0)
- added FB204: 30 Ohms @ 100 MHz, Inductor_SMD:L_0603_1608Metric, F.Cu at (201.8, 112.1)
- added FB205: 30 Ohms @ 100 MHz, Inductor_SMD:L_0603_1608Metric, F.Cu at (229.8, 127.4)
- added FB206: 75 Ohms @ 100 MHz, Inductor_SMD:L_0603_1608Metric, F.Cu at (229.9, 120.9)
- added J305: Conn_Coaxial, Connector_Coaxial:SMA_Amphenol_901-144_Vertical, F.Cu at (63.0, 141.5)
- added J306: Conn_Coaxial, Connector_Coaxial:SMA_Amphenol_901-144_Vertical, F.Cu at (66.0, 30.0)
- added L801: 760 nH, Inductor_SMD:L_Coilcraft_XAL4030-XXX, F.Cu at (242.8, 100.5)
- added R206: 10K, Resistor_SMD:R_0603_1608Metric, F.Cu at (199.0, 75.8)
- added R207: 100k, Resistor_SMD:R_0603_1608Metric, F.Cu at (219.8, 115.7)
- added R208: 100k, Resistor_SMD:R_0603_1608Metric, F.Cu at (206.3, 99.4)
- added R209: 100k, Resistor_SMD:R_0603_1608Metric, F.Cu at (226.0, 116.0)
- added R210: 16K, Resistor_SMD:R_0603_1608Metric, F.Cu at (198.0, 101.2)
- added R211: 10K, Resistor_SMD:R_0603_1608Metric, F.Cu at (198.0, 98.0)
- added R301: 10, Resistor_SMD:R_0603_1608Metric, F.Cu at (63.8, 131.5)
- added R306: 1, Resistor_SMD:R_0603_1608Metric, F.Cu at (102.5, 59.5)
- added R307: 10k, Resistor_SMD:R_0603_1608Metric, F.Cu at (79.0, 87.5)
- added R308: 14.3k 1%, Resistor_SMD:R_0603_1608Metric, F.Cu at (75.0, 76.5)
- added R801: 10, Resistor_SMD:R_0603_1608Metric, F.Cu at (241.8, 97.0)
- added R802: 10, Resistor_SMD:R_0603_1608Metric, F.Cu at (243.8, 104.0)
- added U202: ADP1755ACPZ-R7, Package_CSP:Analog_LFCSP-16-1EP_4x4mm_P0.65mm_EP2.1x2.1mm_ThermalVias, F.Cu at (203.0, 79.7)
- added U203: ADP1755ACPZ-R7, Package_CSP:Analog_LFCSP-16-1EP_4x4mm_P0.65mm_EP2.1x2.1mm_ThermalVias, F.Cu at (201.8, 102.0)
- added U401: 2450BL15B050E, RF:2450BL15B050E_JOT, F.Cu at (60.8, 93.1)
- added U501: 2450BL15B050E, RF:2450BL15B050E_JOT, F.Cu at (62.9, 60.2)
- added U601: 2450BL15B050E, RF:2450BL15B050E_JOT, F.Cu at (60.7, 43.6)
- added U901: 2450BL15B050E, RF:2450BL15B050E_JOT, F.Cu at (63.9, 112.7)
- added Y301: 402F4001XIAR, Crystal:XTAL_402F4001XIAR, F.Cu at (100.2, 79.0)
- C201: renamed from C202; value 0.33uF -> 0.33µF
- C202: renamed from C203; value 1nF -> 22µF
- C203: renamed from C201; value 22uF -> 0.33µF
- C206: renamed from C207; value 8200pF -> 750pF
- C207: renamed from C206; value 750pF -> 1µF
- C208, C209: value C -> 1µF
- C210: renamed from C204; value 100uF -> 1µF; footprint Capacitor_SMD:C_1206_3216Metric -> Capacitor_SMD:C_0603_1608Metric
- C211: renamed from C205; value 0.15uF -> 0.01µF; footprint Capacitor_SMD:C_0603_1608Metric -> Capacitor_SMD:C_0805_2012Metric
- C307: renamed from C301; value 18pF -> 0.001µF
- C308: renamed from C302; value 18pF -> 0.001µF
- C309: renamed from C303; value 18pF -> 1µF
- C310: renamed from C304; value 18pF -> 1µF
- C901: value 4.7uF -> 0.001µF
- C902: value 4.7uF -> 10 µF
- L201: value 250nH -> 270nH; footprint Inductor_SMD:L_12x12mm_H8mm -> Inductor_SMD:L_Coilcraft_XAL4040-XXX
- R201: renamed from R202; value 100k -> 3.01k
- R202: renamed from R201; value 100k -> 60.4k
- R203: value 3.01k -> 100k
- R204: value 60.4k -> 16K
- R303: renamed from R302; value 49R9 -> 10
- R304: renamed from R303; value 10 -> 49R9
- R305: renamed from R304; value 10 -> 1
- moved U201 151.5 mm to (222.6, 109.2), turned to 180 degrees
- moved L201 124.2 mm to (221.6, 102.7), turned to -90 degrees
- moved R202 123.8 mm to (229.5, 113.5), turned to -90 degrees
- moved C201 121.1 mm to (226.9, 107.4), turned to 90 degrees
- moved R201 116.7 mm to (222.0, 118.0), turned to 180 degrees
- moved C203 112.6 mm to (217.8, 107.7), turned to 90 degrees
- moved R205 106.8 mm to (229.5, 116.5), turned to -90 degrees
- moved C202 106.5 mm to (227.8, 107.4), turned to 90 degrees
- moved C206 103.2 mm to (224.3, 115.7), turned to -90 degrees
- moved C902 98.2 mm to (62.5, 117.0), turned to -90 degrees
- moved C901 97.8 mm to (64.0, 117.0), turned to -90 degrees
- moved R203 86.8 mm to (205.2, 75.4), turned to 180 degrees
- moved R302 83.6 mm to (63.8, 133.0), turned to 180 degrees
- moved C305 83.2 mm to (63.8, 130.0), turned to 180 degrees
- moved R204 80.7 mm to (199.0, 78.8), turned to 90 degrees
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- renumbered C306 to C305, C305 to C306, R301 to R302
Connections:
- net Net-(L201-Pad2) renamed /POWER/SW
- C201 pad 1: /POWER/Vin -> /POWER/Vf
- C202 pad 1: /POWER/ss -> /POWER/Vf
- C203 pad 1: /POWER/Vin -> /POWER/Vf
- C206 pad 2: Net-(C207-Pad2) -> AGND
- C207 pad 1: /POWER/Vc -> /POWER/Vdd_GPO
- C208 pad 1: /POWER/Vout -> /POWER/Vdd_GPO
- C208 pad 2: /POWER/Fb -> GND
- C209 pad 1: /POWER/Fb -> /POWER/Vdd_Interface
- C210 pad 1: /POWER/Vout -> /POWER/Vdd_Interface
- C211 pad 1: /POWER/Vout -> /POWER/Vdd_GPO
- C305 pad 1: Net-(C306-Pad1) -> Net-(C305-Pad1)
- C305 pad 2: /RF/TX_MON2 -> /RF/TX_MON1
- C306 pad 1: Net-(C305-Pad1) -> Net-(C306-Pad1)
- C306 pad 2: /RF/TX_MON1 -> /RF/TX_MON2
- C307 pad 1: /RF/SMA/BAL_OUT1 -> /RF/Vdd_RX_VCO
- C307 pad 2: /RF/RX1A_N -> GND
- C308 pad 1: /RF/SMA/BAL_OUT2 -> /RF/Vdd_TX_VCO
- C308 pad 2: /RF/RX1A_P -> GND
- C309 pad 1: /RF/SMA1/BAL_OUT1 -> Net-(C309-Pad1)
- C309 pad 2: /RF/RX2A_N -> GND
- C310 pad 1: /RF/SMA1/BAL_OUT2 -> Net-(C310-Pad1)
- C310 pad 2: /RF/RX2A_P -> GND
- C901 pad 1: /POWER/Vout -> /RF/1P3_TX1A
- C902 pad 1: /POWER/LDO/1V3 -> /RF/1P3_TX1A
- R201 pad 1: /POWER/Pg -> Net-(C205-Pad2)
- R201 pad 2: /POWER/Vout -> AGND
- R202 pad 1: Net-(U201-RT) -> /POWER/Vout
- R202 pad 2: GND -> /POWER/Fb
- R203 pad 1: Net-(C207-Pad2) -> /POWER/VoutX
- R203 pad 2: GND -> /POWER/PG1
- R204 pad 1: /POWER/Vout -> /POWER/1V3A
- R204 pad 2: /POWER/Fb -> Net-(U202-ADJ)
- R205 pad 2: GND -> AGND
- R302 pad 2: Net-(R301-Pad2) -> /RF/TXM1
- R303 pad 1: GND -> /RF/TXM2
- R303 pad 2: Net-(R302-Pad2) -> Net-(C306-Pad1)
- R304 pad 1: Net-(R301-Pad2) -> GND
- R304 pad 2: Net-(C305-Pad1) -> /RF/TXM2
- R305 pad 1: Net-(R302-Pad2) -> Net-(C309-Pad1)
- R305 pad 2: Net-(C306-Pad1) -> /RF/Vdd_RX_VCO
- U201 pad 13: /POWER/Vin -> /POWER/Vf
- U201 pad 14: /POWER/Vin -> /POWER/Vf
- U201 pad 15: /POWER/Vin -> /POWER/Vf
- U201 pad 17: /POWER/Vin -> /POWER/Vf
- U201 pad 18: Net-(U201-RT) -> /POWER/Rt
- U201 pad 3: unconnected-(U201-AGND-Pad3) -> AGND
- U201 pad 4: /POWER/Vin -> /POWER/Vf
- U201 pad 5: /POWER/Vin -> /POWER/Vf
- U201 pad 6: /POWER/Vin -> /POWER/Vf
- U301 pad A1: GND -> /RF/RX2A_N
- U301 pad A10: unconnected-(U301A-TX2B_P-PadA10) -> /RF/1P3_TX2A
- U301 pad A11: unconnected-(U301A-VDDA1P1_TX_VCO-PadA11) -> /RF/Vdd_TX_VCO
- U301 pad A2: GND -> /RF/RX2A_P
- U301 pad A5: unconnected-(U301A-TX_MON2-PadA5) -> /RF/TX_MON2
- U301 pad A7: unconnected-(U301A-TX2A_N-PadA7) -> /RF/TX2A_N
- U301 pad A8: unconnected-(U301A-TX2A_P-PadA8) -> /RF/TX2A_P
- U301 pad A9: unconnected-(U301A-TX2B_N-PadA9) -> /RF/1P3_TX2A
- U301 pad B10: unconnected-(U301A-VDDA1P3_TX_VCO_LDO-PadB10) -> /RF/Vdd_TX_LO
- U301 pad B11: unconnected-(U301A-TX_VCO_LDO_OUT-PadB11) -> /RF/Vdd_TX_VCO
- U301 pad B8: unconnected-(U301A-VDD_GPO-PadB8) -> /RF/Vdd_GPO
- U301 pad B9: unconnected-(U301A-VDDA1P3_TX_LO-PadB9) -> /RF/Vdd_TX_LO
- U301 pad C4: unconnected-(U301A-TEST/ENABLE-PadC4) -> GND
- U301 pad D2: unconnected-(U301A-VDDA1P3_RX_RF-PadD2) -> /RF/Vdd_RX_TX
- U301 pad D3: unconnected-(U301A-VDDA1P3_RX_TX-PadD3) -> /RF/Vdd_RX_TX
- U301 pad E2: unconnected-(U301A-VDDA1P3_RX_LO-PadE2) -> /RF/Vdd_RX_LO
- U301 pad E3: unconnected-(U301A-VDDA1P3_TX_LO_BUFFER-PadE3) -> /RF/Vdd_RX_TX
- U301 pad F12: unconnected-(U301A-VDDD1P3_DIG-PadF12) -> /RF/Vdd_DIG
- U301 pad F2: unconnected-(U301A-VDDA1P3_RX_VCO_LDO-PadF2) -> /RF/Vdd_RX_LO
- U301 pad G2: unconnected-(U301A-RX_VCO_LDO_OUT-PadG2) -> /RF/Vdd_RX_VCO
- U301 pad G3: unconnected-(U301A-VDDA1P1_RX_VCO-PadG3) -> /RF/Vdd_RX_VCO
- U301 pad H12: unconnected-(U301A-VDD_INTERFACE-PadH12) -> /RF/Vdd_Interface
- U301 pad H4: unconnected-(U301A-TXNRX-PadH4) -> /RF/TXnRX
- U301 pad H5: unconnected-(U301A-SYNC_IN-PadH5) -> /RF/SYNCIn
- U301 pad J3: unconnected-(U301A-VDDA1P3_RX_SYNTH-PadJ3) -> /RF/Vdd_RX_SYNTH
- U301 pad K3: unconnected-(U301A-VDDA1P3_TX_SYNTH-PadK3) -> /RF/Vdd_TX_SYNTH
- U301 pad K4: unconnected-(U301A-VDDA1P3_BB-PadK4) -> /RF/Vdd_BB
- U301 pad K5: unconnected-(U301A-RESETB-PadK5) -> Net-(U301A-RESETB)
- U301 pad L4: unconnected-(U301A-RBIAS-PadL4) -> Net-(U301A-RBIAS)
- U301 pad L5: unconnected-(U301A-AUXADC-PadL5) -> /RF/AuxADC
- U301 pad M1: GND -> /RF/RX1A_P
- U301 pad M10: unconnected-(U301A-TX1B_N-PadM10) -> /RF/1P3_TX1A
- U301 pad M11: unconnected-(U301A-XTALP-PadM11) -> Net-(U301A-XTALP)
- U301 pad M12: unconnected-(U301A-XTALN-PadM12) -> Net-(U301A-XTALN)
- U301 pad M2: GND -> /RF/RX1A_N
- U301 pad M5: unconnected-(U301A-TX_MON1-PadM5) -> /RF/TX_MON1
- U301 pad M7: unconnected-(U301A-TX1A_P-PadM7) -> /RF/TX1A_P
- U301 pad M8: unconnected-(U301A-TX1A_N-PadM8) -> /RF/TX1A_N
- U301 pad M9: unconnected-(U301A-TX1B_P-PadM9) -> /RF/1P3_TX1A
Routing:
- net /POWER/Fb: track 0.00 -> 10.3 mm
- net /POWER/Vf: track 0.00 -> 6.65 mm, vias 0 -> 3
- net /POWER/Pg: track 0.00 -> 5.58 mm
- net /POWER/Vc: track 0.00 -> 5.28 mm
- net /POWER/Rt: track 0.00 -> 5.08 mm
- net /POWER/ss: track 0.00 -> 4.19 mm
- net /POWER/Sync: track 0.00 -> 2.43 mm, vias 0 -> 2
- net AGND: track 0.00 -> 1.00 mm, vias 0 -> 6
- net GND: vias 0 -> 10
- net /POWER/Vout: vias 0 -> 11
- added copper zone on F.Cu, net /POWER/SW
- added copper zone on F.Cu, net /POWER/Vf
- added copper zone on F.Cu, net /POWER/Vout
- added copper zone on In5.Cu, net /POWER/Vout
- added copper zone on In6.Cu, net GND
