File: FCOMMS_AD9361/FCOMMS_AD9361.kicad_sch (KiCad schematic)
At the start: 0 parts

Commit message: agile RF
Other:
- sheet POWER ports: added 3A, 3B, PG1, PG2, Vdd_GPO, Vdd_Interface, Vin; removed none
- sheet RF ports: added Vdd_BB, Vdd_DIG, Vdd_GPO, Vdd_Interface, Vdd_RX_LO, Vdd_RX_SYNTH, Vdd_RX_TX, Vdd_RX_VCO, Vdd_TX_LO, Vdd_TX_SYNTH, Vdd_TX_VCO; removed none
- note added: "VDD_GPO must rise as fast or faster than the 1.3 V supply domain"
- note added: "interface in LVDS mode, supply 1.8 V"
