File: FCOMMS_AD9361/LDO.kicad_sch (KiCad schematic)
At the start: 7 parts, among them U1001 ADP1755ACPZ-R7

Commit message: agile RF
Parts:
- added C903: 4.7uF, Capacitor_SMD:C_0805_2012Metric, symbol Device:C
- added C905, C906, C907, C908: 0.1 µF, Capacitor_SMD:C_0603_1608Metric, symbol Device:C
- renumbered C1001 to C901, C903 to C902, C1003 to C904, R902 to R901, R1002 to R902, R1003 to R903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
Connections:
- net 1V3: now also C903.1, C905.1, C906.1, C907.1, C908.1
- net GND: now also C903.2, C905.2, C906.2, C907.2, C908.2
Other:
- moved on the sheet: C904
