File: FCOMMS_AD9361/RF.kicad_sch (KiCad schematic)
At the start: 19 parts, among them J301 Conn_Coaxial, J302 Conn_Coaxial, J303 Conn_Coaxial, J304 Conn_Coaxial, U301 AD9361BBCZ

Commit message: agile RF
Parts:
- removed TP301, TP302, TP303, TP304: TestPoint, TestPoint:TestPoint_Pad_D1.0mm, symbol Connector:TestPoint
- added C307, C308: 0.001µF, Capacitor_SMD:C_0603_1608Metric, symbol Device:C
- added C309, C310: 1µF, Capacitor_SMD:C_0603_1608Metric, symbol Device:C
- added C311: 12pF, Capacitor_SMD:C_0603_1608Metric, symbol Device:C
- added C312: 12 pF, Capacitor_SMD:C_0603_1608Metric, symbol Device:C
- added J305, J306: Conn_Coaxial, Connector_Coaxial:SMA_Amphenol_901-144_Vertical, symbol Connector:Conn_Coaxial
- added R305, R306: 1, Resistor_SMD:R_0603_1608Metric, symbol Device:R
- added R307: 10k, Resistor_SMD:R_0603_1608Metric, symbol Device:R
- added R308: 14.3k 1%, Resistor_SMD:R_0603_1608Metric, symbol Device:R
- added Y301: 402F4001XIAR, 402F4001XIAR:XTAL_402F4001XIAR, symbol 402F4001XIAR:402F4001XIAR
- U301: footprint Package_BGA:BC_144_7_ADI -> BC_144_7_ADI
- renumbered R303 to R301, R301 to R302, R304 to R303, R302 to R304
Connections:
- net GND: now also U301.C4 (TEST/ENABLE), C307.2, C308.2, C309.2, C310.2, C311.2, C312.2, J305.2 (Ext), J306.2 (Ext), R308.1, Y301.2 (GND), Y301.4 (GND__1); no longer U301.A1 (RX2A_N), U301.A2 (RX2A_P), U301.M1 (RX1A_P), U301.M2 (RX1A_N)
- net RX1A_N: now also U301.M2 (RX1A_N)
- net RX1A_P: now also U301.M1 (RX1A_P)
- net RX2A_N: now also U301.A1 (RX2A_N)
- net RX2A_P: now also U301.A2 (RX2A_P)
- net TX1A_N: now also U301.M8 (TX1A_N)
- net TX1A_P: now also U301.M7 (TX1A_P)
- net TX2A_N: now also U301.A7 (TX2A_N)
- net TX2A_P: now also U301.A8 (TX2A_P)
- net TX_MON1: now also U301.M5 (TX_MON1)
- net TX_MON2: now also U301.A5 (TX_MON2)
- net TXM2: now reaches R303.1, R304.2
- net TXM2: now also J306.1 (In)
- net TXM1: now reaches R301.1, R302.2
- net TXM1: now also J305.1 (In)
- net 1P3_TX2A: now reaches U301.A10 (TX2B_P)
- net 1P3_TX2A: now also U301.A9 (TX2B_N)
- net Vdd_TX_VCO: now reaches U301.A11 (VDDA1P1_TX_VCO)
- net Vdd_TX_VCO: now also U301.B11 (TX_VCO_LDO_OUT), C308.1, R306.2
- net Vdd_TX_LO: now reaches U301.B10 (VDDA1P3_TX_VCO_LDO)
- net Vdd_TX_LO: now also U301.B9 (VDDA1P3_TX_LO)
- net Vdd_GPO: now reaches U301.B8 (VDD_GPO)
- net Vdd_RX_TX: now reaches U301.D2 (VDDA1P3_RX_RF)
- net Vdd_RX_TX: now also U301.D3 (VDDA1P3_RX_TX), U301.E3 (VDDA1P3_TX_LO_BUFFER)
- net Vdd_RX_LO: now reaches U301.E2 (VDDA1P3_RX_LO)
- net Vdd_RX_LO: now also U301.F2 (VDDA1P3_RX_VCO_LDO)
- net Vdd_DIG: now reaches U301.F12 (VDDD1P3_DIG)
- net Vdd_RX_VCO: now reaches U301.G2 (RX_VCO_LDO_OUT)
- net Vdd_RX_VCO: now also U301.G3 (VDDA1P1_RX_VCO), C307.1, R305.2
- net Vdd_Interface: now reaches U301.H12 (VDD_INTERFACE)
- net Vdd_Interface: now also R307.2
- net TXnRX: now reaches U301.H4 (TXNRX)
- net SYNCIn: now reaches U301.H5 (SYNC_IN)
- net Vdd_RX_SYNTH: now reaches U301.J3 (VDDA1P3_RX_SYNTH)
- net Vdd_TX_SYNTH: now reaches U301.K3 (VDDA1P3_TX_SYNTH)
- net Vdd_BB: now reaches U301.K4 (VDDA1P3_BB)
- net at U301.K5 (RESETB): now also R307.1
- net at U301.L4 (RBIAS): now also R308.2
- net AuxADC: now reaches U301.L5 (AUXADC)
- net 1P3_TX1A: now reaches U301.M10 (TX1B_N)
- net 1P3_TX1A: now also U301.M9 (TX1B_P)
- net at U301.M11 (XTALP): now also C312.1, Y301.3
- net at U301.M12 (XTALN): now also C311.1, Y301.1
- new net: C309.1, R305.1
- new net: C310.1, R306.1
Other:
- removed sheet SMA2
- removed sheet SMA3
- added sheet SAM_TX (SMAtx.kicad_sch)
- added sheet SAM_TX1 (SMAtx.kicad_sch)
- moved on the sheet: C301, C302, C303, C304, C305, C306, J301, J302, J303, J304, R301, R302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

Commit message: add local library
Parts:
- C301, C302, C303, C304, C305, C306, C307, C308, C309, C310, C311, C312: symbol Device:C -> Library:C
- J301, J302, J303, J304, J305, J306: symbol Connector:Conn_Coaxial -> Library:Conn_Coaxial
- R301, R302, R303, R304, R305, R306, R307, R308: symbol Device:R -> Library:R
- U301: symbol AD9361:AD9361BBCZ -> Library:AD9361BBCZ
- Y301: symbol 402F4001XIAR:402F4001XIAR -> Library:402F4001XIAR
Changed lines of the file:
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@@
 	)
 	(symbol
-		(lib_id "Device:C")
+		(lib_id "Library:C")
 		(at 50.8 137.16 0)
 		(unit 1)
@@
 	)
 	(symbol
-		(lib_id "Device:C")
+		(lib_id "Library:C")
 		(at 109.22 41.91 90)
 		(unit 1)
@@
 	)
 	(symbol
-		(lib_id "power:GND")
+		(lib_id "Library:GND")
 		(at 50.8 50.8 0)
 		(unit 1)
@@
 	)
 	(symbol
-		(lib_id "Device:R")
+		(lib_id "Library:R")
 		(at 359.41 149.86 90)
 		(unit 1)
@@
 	)
 	(symbol
-		(lib_id "power:GND")
+		(lib_id "Library:GND")
 		(at 370.84 154.94 90)
 		(unit 1)
@@
 	)
 	(symbol
-		(lib_id "Device:R")
+		(lib_id "Library:R")
 		(at 78.74 104.14 90)
 		(unit 1)
@@
 	)
 	(symbol
-		(lib_id "AD9361:AD9361BBCZ")
+		(lib_id "Library:AD9361BBCZ")
 		(at 45.72 220.98 0)
 		(unit 2)
@@
 	)
 	(symbol
-		(lib_id "Connector:Conn_Coaxial")
+		(lib_id "Library:Conn_Coaxial")
 		(at 50.8 44.45 0)
 		(mirror y)
@@
 	)
 	(symbol
-		(lib_id "power:GND")
+		(lib_id "Library:GND")
 		(at 38.1 274.32 0)
 		(unit 1)
@@
 	)
 	(symbol
-		(lib_id "Device:C")
+		(lib_id "Library:C")
 		(at 55.88 146.05 0)
 		(unit 1)
@@
 	)
 	(symbol
-		(lib_id "power:GND")
+		(lib_id "Library:GND")
 		(at 114.3 274.32 0)
 		(unit 1)
@@
 	)
 	(symbol
-		(lib_id "Device:R")
+		(lib_id "Library:R")
 		(at 359.41 154.94 270)
 		(unit 1)
@@
 	)
 	(symbol
-		(lib_id "Device:C")
+		(lib_id "Library:C")
 		(at 365.76 219.71 0)
 		(unit 1)
@@
 	)
 	(symbol
-		(lib_id "402F4001XIAR:402F4001XIAR")
+		(lib_id "Library:402F4001XIAR")
 		(at 379.73 208.28 0)
 		(unit 1)
@@
 	)
 	(symbol
-		(lib_id "Device:R")
+		(lib_id "Library:R")
 		(at 63.5 93.98 180)
 		(unit 1)
@@
 	)
 	(symbol
-		(lib_id "Device:C")
+		(lib_id "Library:C")
 		(at 109.22 46.99 90)
 		(unit 1)
@@
 	)
 	(symbol
-		(lib_id "Connector:Conn_Coaxial")
+		(lib_id "Library:Conn_Coaxial")
 		(at 50.8 69.85 0)
 		(mirror y)
@@
 	)
 	(symbol
-		(lib_id "power:GND")
+		(lib_id "Library:GND")
 		(at 50.8 63.5 0)
 		(unit 1)
@@
 	)
 	(symbol
-		(lib_id "power:GND")
+		(lib_id "Library:GND")
 		(at 53.34 152.4 0)
 		(unit 1)
@@
 	)
 	(symbol
-		(lib_id "Device:C")
+		(lib_id "Library:C")
 		(at 95.25 104.14 90)
 		(unit 1)
@@
 	)
 	(symbol
-		(lib_id "power:GND")
+		(lib_id "Library:GND")
 		(at 50.8 38.1 0)
 		(unit 1)
@@
 	)
 	(symbol
-		(lib_id "Device:C")
+		(lib_id "Library:C")
 		(at 76.2 137.16 0)
 		(unit 1)
@@
 	)
 	(symbol
-		(lib_id "Device:C")
+		(lib_id "Library:C")
 		(at 109.22 29.21 90)
 		(unit 1)
@@
 	)
 	(symbol
-		(lib_id "Device:C")
+		(lib_id "Library:C")
 		(at 109.22 34.29 90)
 		(unit 1)
@@
 	)
 	(symbol
-		(lib_id "Device:C")
+		(lib_id "Library:C")
 		(at 96.52 88.9 90)
 		(unit 1)
@@
 	)
 	(symbol
-		(lib_id "Device:C")
+		(lib_id "Library:C")
 		(at 360.68 219.71 0)
 		(unit 1)
@@
 	)
 	(symbol
-		(lib_id "power:GND")
+		(lib_id "Library:GND")
 		(at 363.22 228.6 0)
 		(unit 1)
@@
 	)
 	(symbol
-		(lib_id "power:GND")
+		(lib_id "Library:GND")
 		(at 389.89 217.17 0)
 		(unit 1)
@@
 	)
 	(symbol
-		(lib_id "Connector:Conn_Coaxial")
+		(lib_id "Library:Conn_Coaxial")
 		(at 50.8 88.9 0)
 		(mirror y)
@@
 	)
 	(symbol
-		(lib_id "power:GND")
+		(lib_id "Library:GND")
 		(at 355.6 180.34 90)
 		(unit 1)
@@
 	)
 	(symbol
-		(lib_id "Connector:Conn_Coaxial")
+		(lib_id "Library:Conn_Coaxial")
 		(at 50.8 104.14 0)
 		(mirror y)
@@
 	)
 	(symbol
-		(lib_id "power:GND")
+		(lib_id "Library:GND")
 		(at 63.5 114.3 0)
 		(unit 1)
@@
 	)
 	(symbol
-		(lib_id "power:GND")
+		(lib_id "Library:GND")
 		(at 228.6 247.65 0)
 		(unit 1)
@@
 	)
 	(symbol
-		(lib_id "Device:R")
+		(lib_id "Library:R")
 		(at 81.28 133.35 180)
 		(unit 1)
@@
 	)
 	(symbol
-		(lib_id "Device:R")
+		(lib_id "Library:R")
 		(at 63.5 109.22 180)
 		(unit 1)
@@
 	)
 	(symbol
-		(lib_id "Connector:Conn_Coaxial")
+		(lib_id "Library:Conn_Coaxial")
 		(at 50.8 31.75 0)
 		(mirror y)
@@
 	)
 	(symbol
-		(lib_id "Device:C")
+		(lib_id "Library:C")
 		(at 81.28 146.05 0)
 		(unit 1)
@@
 	)
 	(symbol
-		(lib_id "Device:R")
+		(lib_id "Library:R")
 		(at 55.88 133.35 180)
 		(unit 1)
@@
 	)
 	(symbol
-		(lib_id "Connector:Conn_Coaxial")
+		(lib_id "Library:Conn_Coaxial")
 		(at 50.8 57.15 0)
 		(mirror y)
@@
 	)
 	(symbol
-		(lib_id "power:GND")
+		(lib_id "Library:GND")
 		(at 78.74 152.4 0)
 		(unit 1)
@@
 	)
 	(symbol
-		(lib_id "Device:R")
+		(lib_id "Library:R")
 		(at 76.2 88.9 90)
 		(unit 1)
@@
 	)
 	(symbol
-		(lib_id "power:GND")
+		(lib_id "Library:GND")
 		(at 50.8 76.2 0)
 		(unit 1)
@@
 	)
 	(symbol
-		(lib_id "AD9361:AD9361BBCZ")
+		(lib_id "Library:AD9361BBCZ")
 		(at 233.68 38.1 0)
 		(unit 1)
@@
 	)
 	(symbol
-		(lib_id "power:GND")
+		(lib_id "Library:GND")
 		(at 63.5 99.06 0)
 		(unit 1)
