File: FCOMMS_AD9361/SMAtx.kicad_sch (KiCad schematic)
At the start: 3 parts, among them U601 2450BL15B050E

Commit message: add local library
Parts:
- C601, C602: symbol Device:C -> Library:C
- U601: symbol 2.45GHz_Balun:2450BL15B050E -> Library:2450BL15B050E
Changed lines of the file:
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@@
 	)
 	(symbol
-		(lib_id "Device:C")
+		(lib_id "Library:C")
 		(at 106.68 109.22 0)
 		(unit 1)
@@
 	)
 	(symbol
-		(lib_id "power:GND")
+		(lib_id "Library:GND")
 		(at 199.39 85.09 90)
 		(unit 1)
@@
 	)
 	(symbol
-		(lib_id "power:GND")
+		(lib_id "Library:GND")
 		(at 96.52 119.38 0)
 		(unit 1)
@@
 	)
 	(symbol
-		(lib_id "2.45GHz_Balun:2450BL15B050E")
+		(lib_id "Library:2450BL15B050E")
 		(at 113.03 82.55 0)
 		(unit 1)
@@
 	)
 	(symbol
-		(lib_id "Device:C")
+		(lib_id "Library:C")
 		(at 91.44 109.22 0)
 		(unit 1)
