File: FCOMMS_AD9361/emi.kicad_sch (KiCad schematic)
At the start: 6 parts

Commit message: add local library
Parts:
- C801, C802, C803: symbol Device:C -> Library:C
- L801: symbol Device:L -> Library:L
- R801, R802: symbol Device:R -> Library:R
Changed lines of the file:
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@@
 	)
 	(symbol
-		(lib_id "Device:C")
+		(lib_id "Library:C")
 		(at 127 76.2 0)
 		(unit 1)
@@
 	)
 	(symbol
-		(lib_id "Device:C")
+		(lib_id "Library:C")
 		(at 177.8 76.2 0)
 		(unit 1)
@@
 	)
 	(symbol
-		(lib_id "Device:C")
+		(lib_id "Library:C")
 		(at 152.4 99.06 0)
 		(unit 1)
@@
 	)
 	(symbol
-		(lib_id "Device:L")
+		(lib_id "Library:L")
 		(at 165.1 50.8 90)
 		(unit 1)
@@
 	)
 	(symbol
-		(lib_id "Device:R")
+		(lib_id "Library:R")
 		(at 127 102.87 0)
 		(unit 1)
@@
 	)
 	(symbol
-		(lib_id "power:GND")
+		(lib_id "Library:GND")
 		(at 152.4 130.81 0)
 		(unit 1)
@@
 	)
 	(symbol
-		(lib_id "Device:R")
+		(lib_id "Library:R")
 		(at 177.8 100.33 0)
 		(unit 1)
