File: FCOMMS_AD9361/sma.kicad_sch (KiCad schematic)
At the start: 1 part, among them U401 2450BL15B050E

Commit message: add local library
Parts:
- U401: symbol 2.45GHz_Balun:2450BL15B050E -> Library:2450BL15B050E
Changed lines of the file:
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@@
 	)
 	(symbol
-		(lib_id "power:GND")
+		(lib_id "Library:GND")
 		(at 88.9 83.82 270)
 		(unit 1)
@@
 	)
 	(symbol
-		(lib_id "power:GND")
+		(lib_id "Library:GND")
 		(at 179.07 83.82 90)
 		(unit 1)
@@
 	)
 	(symbol
-		(lib_id "2.45GHz_Balun:2450BL15B050E")
+		(lib_id "Library:2450BL15B050E")
 		(at 92.71 81.28 0)
 		(unit 1)
